File: rf_gateway.sch (KiCad schematic (older format))
At the start: 7 parts, among them J101 PJ-202A, J102 Conn_01x03_Female, J103 Conn_01x05_Male, U101 ESP32-WROOM-32

Commit message: First RC
Parts:
- removed J101: PJ-202A, digikey-footprints:Barrel_Jack_5.5mmODx2.1mmID_PJ-202A, symbol dk_Barrel-Power-Connectors:PJ-202A
- removed J102: Conn_01x03_Female, Connector_JST:JST_EH_B3B-EH-A_1x03_P2.50mm_Vertical, symbol Connector:Conn_01x03_Female
- removed J103: Conn_01x05_Male, Connector_JST:JST_EH_B5B-EH-A_1x05_P2.50mm_Vertical, symbol Connector:Conn_01x05_Male
- removed U101: ESP32-WROOM-32, RF_Module:ESP32-WROOM-32, symbol RF_Module:ESP32-WROOM-32
- added C101, C105, C107, C108: 100nF, Capacitor_SMD:C_0805_2012Metric_Pad1.15x1.40mm_HandSolder, symbol Device:C
- added C102, C103: 7pF, Capacitor_SMD:C_0805_2012Metric_Pad1.15x1.40mm_HandSolder, symbol Device:C
- added C104, C106, C110: 10uF, Capacitor_SMD:C_0805_2012Metric_Pad1.15x1.40mm_HandSolder, symbol Device:C
- added C109: 100uF, custom-lib:TAJB107M010RNJ, symbol Device:CP
- added D102: BLUE, LED_SMD:LED_0805_2012Metric_Pad1.15x1.40mm_HandSolder, symbol Device:LED
- added J101: Antena, Connector_PinHeader_2.54mm:PinHeader_1x01_P2.54mm_Vertical, symbol Connector:Conn_01x01_Female
- added L101: 8 Turns, Inductor_THT:L_Axial_L5.3mm_D2.2mm_P7.62mm_Horizontal_Vishay_IM-1, symbol Device:L
- added L102: 3 Turns, Inductor_THT:L_Axial_L5.3mm_D2.2mm_P7.62mm_Horizontal_Vishay_IM-1, symbol Device:L
- added Q101: 2SC3357-T1-A, Package_TO_SOT_SMD:SOT-89-3_Handsoldering, symbol Device:Q_NPN_BCE
- added Q102: S8050, Package_TO_SOT_SMD:SOT-23, symbol Device:Q_NPN_BCE
- added Q103, Q104: Q_NPN_BCE, custom-lib:SOT-523, symbol Device:Q_NPN_BCE
- added R103: 27k, digikey-footprints:0805, symbol Device:R
- added R104, R105: 1k, digikey-footprints:0805, symbol Device:R
- added R106, R107: 10k, digikey-footprints:0805, symbol Device:R
- added U101: TPS3839, Package_TO_SOT_SMD:SOT-23, symbol custom-lib:TPS3839
- added U102: ESP-32s, custom-lib:ESP-32S, symbol custom-lib:ESP-32s
- added U103: C167321, custom-lib:C167321, symbol custom-lib:C167321
- added U104: HT7333-A, Package_TO_SOT_SMD:SOT-89-3_Handsoldering, symbol custom-lib:HT7333-A
- added U105: CH340E, custom-lib:CH340E-MSOP-10, symbol custom-lib:CH340E
- added Y101: 433MHz, custom-lib:C2280, symbol Device:Crystal_GND3
- D101: value LED -> RED; footprint Diode_SMD:D_0805_2012Metric -> LED_SMD:LED_0805_2012Metric_Pad1.15x1.40mm_HandSolder
- R102: value 500 -> 27k
Connections:
- net labels added: +5V, D+, D-, RF, ~CTS, ~RTS
- wire segments 27 -> 105
- no-connect marks 28 -> 32
